File: stm32_test_board.kicad_pcb (KiCad board)
At the start: 2 copper layers, 152 x 116 mm, 125 parts, among them J1 USART1, J10 I2C2, J11 SPI1, J12 LEDS1, J13 LEDS1, J14 SPI2, J15 Conn_02x16_Odd_Even, J16 USB_B, J17 USB Conn, J18 Buttons, J19 Conn_02x20_Odd_Even, J2 Power IN, J20 LEDS1, J21 LEDS1, J22 SWD, J23 VCC, J24 GND, J25 GND, J26 5V, J27 GND, J28 GND, J29 GND, J3 TP1, J30 BAT, J31 VBAT Selector, J32 USB Conn, J4 TP2, J5 USART2, J6 BOOT, J7 USART3, J8 Power Selector, J9 I2C1, Q1 IRLML5203, SW1 Reset, SW2 Reset, SW3 Reset, SW4 Reset, SW5 Reset, U1 AMS1117-3.3, U2 STM32F103C8Tx, Y1 8 MHz, Y2 Crystal

Commit message: Fix some errors
Parts:
- moved L2 1.65 mm to (68.9, 34.1)
- moved C12 1.55 mm to (83.3, 13.8)
- moved C15 1.19 mm to (68.9, 29.1)
- moved C13 1.03 mm to (68.9, 31.7)
Connections:
- J19 pad 13: /PA15 -> /PB3
- J19 pad 14: /PA15 -> /PB3
- J19 pad 15: /PA14 -> /PA15
- J19 pad 16: /PA14 -> /PA15
- J19 pad 17: /PA13 -> /PA14
- J19 pad 18: /PA13 -> /PA14
- J19 pad 19: /PA12 -> /PA13
- J19 pad 20: /PA12 -> /PA13
- J19 pad 21: /PA11 -> /PA12
- J19 pad 22: /PA11 -> /PA12
- J19 pad 23: /PA10 -> /PA11
- J19 pad 24: /PA10 -> /PA11
- J19 pad 25: /PA9 -> /PA10
- J19 pad 26: /PA9 -> /PA10
- J19 pad 27: /PA8 -> /PA9
- J19 pad 28: /PA8 -> /PA9
- J19 pad 29: /PB15 -> /PA8
- J19 pad 30: /PB15 -> /PA8
- J19 pad 31: /PB14 -> /PB15
- J19 pad 32: /PB14 -> /PB15
- J19 pad 33: /PB13 -> /PB14
- J19 pad 34: /PB13 -> /PB14
- J19 pad 35: /PB12 -> /PB13
- J19 pad 36: /PB12 -> /PB13
- J19 pad 37: unconnected-(J19-Pad37) -> /PB12
- J19 pad 38: unconnected-(J19-Pad38) -> /PB12
- J20 pad 13: /PA15 -> /PB3
- J20 pad 15: /PA14 -> /PA15
- J20 pad 17: /PA13 -> /PA14
- J20 pad 19: unconnected-(J20-Pad19) -> /PA13
Routing:
- net /PB3: track 0.00 -> 44.5 mm
- net /PA14: track 81.3 -> 86.8 mm
- net +3V3: track 547.8 -> 542.8 mm
- net /PA12: track 151.7 -> 147.2 mm
- net /PA11: track 141.4 -> 137.6 mm
- net /PB12: track 153.7 -> 150.0 mm
- net /PB7: track 124.6 -> 127.0 mm
- net /PC14: track 61.7 -> 64.0 mm
- net /PC15: track 60.5 -> 62.8 mm
- net /PA15: track 42.3 -> 44.5 mm
- net /PB13: track 90.2 -> 88.1 mm
- net /PA8: track 86.4 -> 84.6 mm
- net /PA10: track 99.8 -> 98.1 mm
- net /PA9: track 92.5 -> 90.9 mm
- net /PB14: track 95.3 -> 93.7 mm
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Other:
- board text added: "PB3"
