File: stm32_test_board.kicad_sch (KiCad schematic)
At the start: 125 parts, among them J1 USART1, J10 I2C2, J11 SPI1, J12 LEDS1, J13 LEDS1, J14 SPI2, J15 Conn_02x16_Odd_Even, J16 USB_B, J17 USB Conn, J18 Buttons, J19 Conn_02x20_Odd_Even, J2 Power IN, J20 LEDS1, J21 LEDS1, J22 SWD, J23 VCC, J24 GND, J25 GND, J26 5V, J27 GND, J28 GND, J29 GND, J3 TP1, J30 BAT, J31 VBAT Selector, J32 USB Conn, J4 TP2, J5 USART2, J6 BOOT, J7 USART3, J8 Power Selector, J9 I2C1, Q1 IRLML5203, SW1 Reset, SW2 Reset, SW3 Reset, SW4 Reset, SW5 Reset, U1 AMS1117-3.3, U2 STM32F103C8Tx, Y1 8 MHz, Y2 Crystal

Commit message: Fix some errors
Parts:
- J32: value USB Conn -> OSC32 Conn
Connections:
- net PA10: now also J19.25 (Pin_25), J19.26 (Pin_26); no longer J19.23 (Pin_23), J19.24 (Pin_24)
- net PA11: now also J19.23 (Pin_23), J19.24 (Pin_24); no longer J19.21 (Pin_21), J19.22 (Pin_22)
- net PA12: now also J19.21 (Pin_21), J19.22 (Pin_22); no longer J19.19 (Pin_19), J19.20 (Pin_20)
- net PA13: now also J19.19 (Pin_19), J19.20 (Pin_20), J20.19 (Pin_19); no longer J19.17 (Pin_17), J19.18 (Pin_18), J20.17 (Pin_17)
- net PA14: now also J19.17 (Pin_17), J19.18 (Pin_18), J20.17 (Pin_17); no longer J19.15 (Pin_15), J19.16 (Pin_16), J20.15 (Pin_15)
- net PA15: now also J19.15 (Pin_15), J19.16 (Pin_16), J20.15 (Pin_15); no longer J19.13 (Pin_13), J19.14 (Pin_14), J20.13 (Pin_13)
- net PA8: now also J19.29 (Pin_29), J19.30 (Pin_30); no longer J19.27 (Pin_27), J19.28 (Pin_28)
- net PA9: now also J19.27 (Pin_27), J19.28 (Pin_28); no longer J19.25 (Pin_25), J19.26 (Pin_26)
- net PB12: now also J19.37 (Pin_37), J19.38 (Pin_38); no longer J19.35 (Pin_35), J19.36 (Pin_36)
- net PB13: now also J19.35 (Pin_35), J19.36 (Pin_36); no longer J19.33 (Pin_33), J19.34 (Pin_34)
- net PB14: now also J19.33 (Pin_33), J19.34 (Pin_34); no longer J19.31 (Pin_31), J19.32 (Pin_32)
- net PB15: now also J19.31 (Pin_31), J19.32 (Pin_32); no longer J19.29 (Pin_29), J19.30 (Pin_30)
- net PB3: now also J19.13 (Pin_13), J19.14 (Pin_14), J20.13 (Pin_13)
- no-connect marks 9 -> 6
